File: BUILD/BUILD.kicad_sch (KiCad schematic)
At the start: 18 parts, among them J1-INPUT1 AudioJack3, SW1 SW_Push, SW2 SW_Push, SW3 SW_DIP_x04, SW4 SW_Push, U2 ADC081C021CIMM

Commit message: 2025-06-19-01
Parts:
- removed U2: ADC081C021CIMM, Package_SO:MSOP-8_3x3mm_P0.65mm, symbol Analog_ADC:ADC081C021CIMM
- added C1, C3, C4, C6: 10uF, symbol Device:C
- added C2, C5: 0.05uF, symbol Device:C
- added J1-OUTPUT, J1-OUTPUT1: AudioJack3, symbol Connector_Audio:AudioJack3
- added R10, R12: 100ohm, symbol Device:R
- added R11, R9: 100Ohm, symbol Device:R
- added R4, R5, R6, R7, R8: 1K, symbol Device:R
- added RV1-Headphone_VOL, RV1-Headphone_VOL1: R_Potentiometer, symbol Device:R_Potentiometer
- added SW5-F1, SW6-F2, SW7-F3, SW8-F4, SW9-F5: SW_Push, symbol Switch:SW_Push
- added U1, U2: LM386, symbol Amplifier_Audio:LM386
- renumbered DS1 to DS1-2x16_LCD
Connections:
- net +5V: now also SW3.5, SW3.6, R4.1; no longer A1.5 (+5V)
- net GND: now also BZ1.2 (-), D1-MRS.1 (K), C4.2, C6.2, J1-OUTPUT.GND, J1-OUTPUT1.GND, R11.2, R9.2, RV1-Headphone_VOL.3, RV1-Headphone_VOL1.3, SW5-F1.1, SW6-F2.1, SW7-F3.1, SW8-F4.1, SW9-F5.1, U1.2 (-), U1.4 (GND), U2.2 (-), U2.4 (GND); no longer A1.6 (GND), J1-INPUT1.GND, SW3.5, SW3.6, SW3.7, SW3.8
- net at A1.14 (SCL/A5): now also R4.2, R5.1, SW5-F1.2
- net at A1.23 (D8): now also SW3.7; no longer BZ1.1 (+)
- net at A1.25 (D10): now also SW3.8; no longer R2.2
- net at A1.28 (D13): now also RV1-Headphone_VOL.1, RV1-Headphone_VOL1.1
- net at A1.31 (SDA/A4): now also A1.32 (SCL/A5)
- net at SW3.2: now also BZ1.1 (+); no longer D1-MRS.1 (K)
- net at SW3.1: now also R2.2; no longer BZ1.2 (-)
- net at SW3.3: now also U1.6 (V+)
- net at SW3.4: now also U2.6 (V+)
- new net: RV1-Headphone_VOL.2, U1.3 (+)
- new net: C2.1, R10.2, U1.5
- new net: C2.2, R9.1
- new net: J1-OUTPUT.L, J1-OUTPUT.R, R10.1
- new net: R5.2, R6.1, SW6-F2.2
- new net: J1-OUTPUT1.L, J1-OUTPUT1.R, R12.1
- new net: C5.1, R12.2, U2.5
- new net: R6.2, R7.1, SW7-F3.2
- new net: R8.2, SW9-F5.2
- new net: C1.1, U1.1 (GAIN)
- new net: C4.1, U1.7 (BYPASS)
- new net: C1.2, U1.8 (GAIN)
- new net: C5.2, R11.1
- new net: R7.2, R8.1, SW8-F4.2
- new net: C6.1, U2.7 (BYPASS)
- new net: C3.1, U2.1 (GAIN)
- new net: C3.2, U2.8 (GAIN)
- new net: RV1-Headphone_VOL1.2, U2.3 (+)
- no-connect marks 1 -> 5
Other:
- moved on the sheet: A1, BZ1, D1-MRS, D2-PWR, DS1-2x16_LCD, J1-INPUT1, R1, R2, R3, RV1-Contrast, RV2-Buzzur_TONE, RV2-Buzzur_VOL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

Commit message: 2025-06-22-05
Parts:
- SW1: value SW_Push -> SW_Push-MODE
- SW2: value SW_Push -> SW_Push-CLEAR
- SW4: value SW_Push -> SW_Push-RESET
Other:
- moved on the sheet: SW1
Changed lines of the file:
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@@
 	)
 	(junction
-		(at 35.56 69.85)
-		(diameter 0)
-		(color 0 0 0 0)
-	)
-	(junction
 		(at 33.02 153.67)
 		(diameter 0)
@@
 	)
 	(junction
+		(at 34.29 69.85)
+		(diameter 0)
+		(color 0 0 0 0)
+	)
+	(junction
 		(at 77.47 87.63)
 		(diameter 0)
@@
 	(wire
 		(pts
-			(xy 180.34 72.39) (xy 45.72 72.39)
+			(xy 180.34 72.39) (xy 53.34 72.39)
 		)
 		(stroke
@@
 	(wire
 		(pts
-			(xy 109.22 116.84) (xy 109.22 113.03)
+			(xy 53.34 80.01) (xy 49.53 80.01)
 		)
 		(stroke
@@
 	(wire
 		(pts
-			(xy 220.98 152.4) (xy 217.17 152.4)
+			(xy 109.22 116.84) (xy 109.22 113.03)
 		)
 		(stroke
@@
 	(wire
 		(pts
-			(xy 157.48 176.53) (xy 157.48 177.8)
+			(xy 220.98 152.4) (xy 217.17 152.4)
 		)
 		(stroke
@@
 	(wire
 		(pts
-			(xy 77.47 133.35) (xy 88.9 133.35)
+			(xy 157.48 176.53) (xy 157.48 177.8)
 		)
 		(stroke
@@
 	(wire
 		(pts
-			(xy 35.56 69.85) (xy 46.99 69.85)
+			(xy 77.47 133.35) (xy 88.9 133.35)
 		)
 		(stroke
@@
 	(wire
 		(pts
-			(xy 29.21 69.85) (xy 35.56 69.85)
+			(xy 29.21 69.85) (xy 34.29 69.85)
 		)
 		(stroke
@@
 	(wire
 		(pts
-			(xy 35.56 80.01) (xy 35.56 69.85)
-		)
-		(stroke
-			(width 0)
-			(type default)
-		)
-	)
-	(wire
-		(pts
 			(xy 111.76 113.03) (xy 111.76 133.35)
 		)
@@
 	(wire
 		(pts
+			(xy 39.37 80.01) (xy 34.29 80.01)
+		)
+		(stroke
+			(width 0)
+			(type default)
+		)
+	)
+	(wire
+		(pts
 			(xy 144.78 148.59) (xy 144.78 151.13)
 		)
@@
 	(wire
 		(pts
+			(xy 34.29 69.85) (xy 34.29 80.01)
+		)
+		(stroke
+			(width 0)
+			(type default)
+		)
+	)
+	(wire
+		(pts
 			(xy 191.77 127) (xy 191.77 118.11)
 		)
@@
 	(wire
 		(pts
-			(xy 45.72 72.39) (xy 45.72 80.01)
+			(xy 34.29 69.85) (xy 46.99 69.85)
+		)
+		(stroke
+			(width 0)
+			(type default)
+		)
+	)
+	(wire
+		(pts
+			(xy 53.34 72.39) (xy 53.34 80.01)
 		)
 		(stroke
@@
 			)
 		)
-		(property "Value" "SW_Push"
+		(property "Value" "SW_Push-RESET"
 			(at 175.26 30.48 0)
 			(effects
@@
 	(symbol
 		(lib_id "Switch:SW_Push")
-		(at 40.64 80.01 0)
+		(at 44.45 80.01 0)
 		(unit 1)
 		(exclude_from_sim no)
@@
 		(fields_autoplaced yes)
 		(property "Reference" "SW1"
-			(at 40.64 72.39 0)
+			(at 44.45 72.39 0)
 			(effects
 				(font
@@
 			)
 		)
-		(property "Value" "SW_Push"
-			(at 40.64 74.93 0)
+		(property "Value" "SW_Push-MODE"
+			(at 44.45 74.93 0)
 			(effects
 				(font
@@
 		)
 		(property "Footprint" ""
-			(at 40.64 74.93 0)
+			(at 44.45 74.93 0)
 			(effects
 				(font
@@
 		)
 		(property "Datasheet" "~"
-			(at 40.64 74.93 0)
+			(at 44.45 74.93 0)
 			(effects
 				(font
@@
 		)
 		(property "Description" "Push button switch, generic, two pins"
-			(at 40.64 80.01 0)
+			(at 44.45 80.01 0)
 			(effects
 				(font
@@
 			)
 		)
-		(property "Value" "SW_Push"
+		(property "Value" "SW_Push-CLEAR"
 			(at 52.07 64.77 0)
 			(effects
